File: hw/ea01/leds.kicad_sch (KiCad schematic)
At the start: 36 parts, among them Q1 BC817, Q2 BC817, Q3 BC817, Q4 BC817, Q5 BC817, Q6 BC817, Q7 BC817

Commit message: schmatic drawing continue...
Connections:
- net OUT_LED renamed OUT1_LED
Changed lines of the file:
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@@
 		)
 	)
-	(global_label "OUT_LED"
+	(global_label "OUT1_LED"
 		(shape input)
 		(at 209.55 71.12 180)
@@
 		)
 		(property "Intersheetrefs" "${INTERSHEET_REFS}"
-			(at 198.5215 71.12 0)
+			(at 197.312 71.12 0)
 			(effects
 				(font
