File: hw/ea01/leds.kicad_sch (KiCad schematic)
At the start: 36 parts, among them Q1 BC817, Q2 BC817, Q3 BC817, Q4 BC817, Q5 BC817, Q6 BC817, Q7 BC817

Commit message: errors fix for comp fp
Parts:
- BZ1: footprint (none) -> Buzzer_Beeper:Buzzer_15x7.5RM7.6
Changed lines of the file:
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@@
 			)
 		)
-		(property "Footprint" ""
+		(property "Footprint" "Buzzer_Beeper:Buzzer_15x7.5RM7.6"
 			(at 67.945 104.14 90)
 			(effects

Commit message: component placement continue..
Parts:
- removed BZ1: Buzzer, Buzzer_Beeper:Buzzer_15x7.5RM7.6, symbol Device:Buzzer
- removed D10, D11, D12, D13, D7, D9: RED_LED, Resistor_SMD:R_0805_2012Metric, symbol Device:LED
- added J13, J14, J15, J16, J17, J18, J6: Conn_01x02_Pin, Connector_PinHeader_2.54mm:PinHeader_1x02_P2.54mm_Vertical, symbol Connector:Conn_01x02_Pin
Connections:
- net +3.3V: now also J13.2 (Pin_2), J14.2 (Pin_2), J15.2 (Pin_2), J16.2 (Pin_2), J17.2 (Pin_2), J18.2 (Pin_2)
- net +6.8V: now also J6.2 (Pin_2)
- net at R25.1: now also J13.1 (Pin_1)
- net at R31.1: now also J15.1 (Pin_1)
- net at R28.1: now also J14.1 (Pin_1)
- net at D8.2 (A), R18.1: now also J6.1 (Pin_1)
- net at R37.1: now also J16.1 (Pin_1)
- net at R17.1: now also J18.1 (Pin_1)
- net at R34.1: now also J17.1 (Pin_1)

Commit message: placement continue...
Parts:
- J13, J14, J15, J16, J17, J18, J6: footprint Connector_PinHeader_2.54mm:PinHeader_1x02_P2.54mm_Vertical -> Connector_PinHeader_1.27mm:PinHeader_1x02_P1.27mm_Vertical
Changed lines of the file:
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@@
 			)
 		)
-		(property "Footprint" "Connector_PinHeader_2.54mm:PinHeader_1x02_P2.54mm_Vertical"
+		(property "Footprint" "Connector_PinHeader_1.27mm:PinHeader_1x02_P1.27mm_Vertical"
 			(at 134.62 34.29 0)
 			(effects
@@
 			)
 		)
-		(property "Footprint" "Connector_PinHeader_2.54mm:PinHeader_1x02_P2.54mm_Vertical"
+		(property "Footprint" "Connector_PinHeader_1.27mm:PinHeader_1x02_P1.27mm_Vertical"
 			(at 201.93 110.49 0)
 			(effects
@@
 			)
 		)
-		(property "Footprint" "Connector_PinHeader_2.54mm:PinHeader_1x02_P2.54mm_Vertical"
+		(property "Footprint" "Connector_PinHeader_1.27mm:PinHeader_1x02_P1.27mm_Vertical"
 			(at 200.66 33.02 0)
 			(effects
@@
 			)
 		)
-		(property "Footprint" "Connector_PinHeader_2.54mm:PinHeader_1x02_P2.54mm_Vertical"
+		(property "Footprint" "Connector_PinHeader_1.27mm:PinHeader_1x02_P1.27mm_Vertical"
 			(at 132.08 107.95 0)
 			(effects
@@
 			)
 		)
-		(property "Footprint" "Connector_PinHeader_2.54mm:PinHeader_1x02_P2.54mm_Vertical"
+		(property "Footprint" "Connector_PinHeader_1.27mm:PinHeader_1x02_P1.27mm_Vertical"
 			(at 264.16 109.22 0)
 			(effects
@@
 			)
 		)
-		(property "Footprint" "Connector_PinHeader_2.54mm:PinHeader_1x02_P2.54mm_Vertical"
+		(property "Footprint" "Connector_PinHeader_1.27mm:PinHeader_1x02_P1.27mm_Vertical"
 			(at 262.89 33.02 0)
 			(effects
@@
 			)
 		)
-		(property "Footprint" "Connector_PinHeader_2.54mm:PinHeader_1x02_P2.54mm_Vertical"
+		(property "Footprint" "Connector_PinHeader_1.27mm:PinHeader_1x02_P1.27mm_Vertical"
 			(at 73.66 107.95 0)
 			(effects

Commit message: placement completed.
Connections:
- net +6.8V renamed +5V
Changed lines of the file:
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@@
 			)
 		)
-		(property "Value" "+6.8V"
+		(property "Value" "+5V"
 			(at 62.23 90.17 0)
 			(effects

Commit message: drawing continue..
Parts:
- removed D8: 1N4148W, Diode_SMD:D_SOD-123, symbol Diode:1N4148W
- removed J6: Conn_01x02_Pin, Connector_PinHeader_1.27mm:PinHeader_1x02_P1.27mm_Vertical, symbol Connector:Conn_01x02_Pin
- removed Q1: BC817, Package_TO_SOT_SMD:SOT-23, symbol Transistor_BJT:BC817
- removed R18, R19: 100R, Resistor_SMD:R_0603_1608Metric, symbol Device:R
- removed R20: 10K, Resistor_SMD:R_0603_1608Metric, symbol Device:R
