File: hw/ea01/mcu.kicad_sch (KiCad schematic)
At the start: 34 parts, among them J2 USB_B, J3 Conn_01x05_Pin, SW1 SW_Push, SW2 SW_Push, U1 RP2040, U11 W25Q32JVSS, U3 NUP2202, Y1 12Mhz

Commit message: schmatic drawing continue...
Parts:
- added C60: 100nF, Capacitor_SMD:C_0603_1608Metric, symbol Device:C
- added C61: 22pF, Capacitor_SMD:C_0603_1608Metric, symbol Device:C
- added J8, J9: Conn_01x03_Pin, symbol Connector:Conn_01x03_Pin
- added R58: 1K, Resistor_SMD:R_0603_1608Metric, symbol Device:R
- added R59: 22R, Resistor_SMD:R_0603_1608Metric, symbol Device:R
- added TP23, TP6, TP7, TP8: TestPoint, TestPoint:TestPoint_Pad_D1.5mm, symbol Connector:TestPoint
Connections:
- net +1.1V: now also TP6.1
- net +3.3V: now also J9.3 (Pin_3), R59.2, TP8.1; no longer U1.43 (ADC_AVDD)
- net GND: now also C60.2, C61.2, J8.1 (Pin_1), J9.1 (Pin_1)
- net RUN: now also TP7.1
- net UART0_RX: now also U1.12 (GPIO9), J8.2 (Pin_2); no longer U1.13 (GPIO10)
- net UART0_TX: now also U1.11 (GPIO8), J8.3 (Pin_3); no longer U1.12 (GPIO9)
- net RS485_TX: now reaches U1.15 (GPIO12)
- net RS485_RX: now reaches U1.16 (GPIO13)
- net RS485_RW: now reaches U1.17 (GPIO14)
- net VIN_MONITOR: now reaches U1.38 (GPIO26_ADC0)
- net ADC_TEST: now reaches U1.39 (GPIO27_ADC1)
- net ADC_TEST: now also C60.1, C61.1, R58.1, TP23.1
- new net: R59.1, U1.43 (ADC_AVDD)
- new net: J9.2 (Pin_2), R58.2
