File: hw/ea01/rtc.kicad_sch (KiCad schematic)
At the start: 2 parts, among them U2 PCF8563T, U8 CAT24C256

Commit message: schmatic drawing continue...
Parts:
- added BT1: Battery_Cell, symbol Device:Battery_Cell
- added C53, C54: 15pF, Capacitor_SMD:C_0603_1608Metric, symbol Device:C
- added C55, C57: 220nF, Capacitor_SMD:C_0603_1608Metric, symbol Device:C
- added C56: 22pF, Capacitor_SMD:C_0603_1608Metric, symbol Device:C
- added D16, D17: SS16, Diode_SMD:D_SMA, symbol Diode:SS16
- added R56: 10K, Resistor_SMD:R_0603_1608Metric, symbol Device:R
- added R57: 1K, Resistor_SMD:R_0603_1608Metric, symbol Device:R
- added TP1, TP2, TP3, TP4, TP5: TestPoint, TestPoint:TestPoint_Pad_D1.5mm, symbol Connector:TestPoint
- added Y2: 32.768Khz, symbol Device:Crystal
Connections:
- net I2C0_SCL: now also U2.6 (SCL), U8.6 (SCL), TP4.1
- net I2C0_SDA: now also U2.5 (SDA), U8.5 (SDA), TP5.1
- net GND: now reaches U8.1 (A0)
- net GND: now also U2.4 (VSS), U8.2 (A1), U8.3 (A2), U8.4 (GND), BT1.2 (-), C53.1, C54.1, C55.2, C56.1, C57.2, R57.1
- net at U8.7 (WP): now also R57.2
- net +3.3V: now reaches U8.8 (VCC)
- net +3.3V: now also C57.1, D16.2 (A), R56.2
- net at U2.1 (OSCI): now also C53.2, Y2.2
- net at U2.2 (OSCO): now also C54.2, Y2.1
- net RTC_INT: now reaches U2.3 (~{INT})
- net RTC_INT: now also R56.1
- net at U2.7 (CLKO): now also TP1.1
- net at U2.8 (VDD): now also C55.1, C56.2, D16.1 (K), D17.1 (K), TP3.1
- new net: BT1.1 (+), D17.2 (A), TP2.1
Other:
- company: (none) -> Enis ASLAN
- title: (none) -> RTC & EEPROM
- moved on the sheet: U2, U8

Commit message: errors fix for comp fp
Parts:
- BT1: footprint (none) -> Connector_PinHeader_2.54mm:PinHeader_1x02_P2.54mm_Vertical
- U8: footprint (none) -> Package_SO:SOIC-8_3.9x4.9mm_P1.27mm
- Y2: footprint (none) -> Crystal:Crystal_C38-LF_D3.0mm_L8.0mm_Horizontal_1EP_style1
Changed lines of the file:
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@@
 			)
 		)
-		(property "Footprint" ""
+		(property "Footprint" "Package_SO:SOIC-8_3.9x4.9mm_P1.27mm"
 			(at 207.01 97.79 0)
 			(effects
@@
 			)
 		)
-		(property "Footprint" ""
+		(property "Footprint" "Connector_PinHeader_2.54mm:PinHeader_1x02_P2.54mm_Vertical"
 			(at 147.32 74.676 90)
 			(effects
@@
 			)
 		)
-		(property "Footprint" ""
+		(property "Footprint" "Crystal:Crystal_C38-LF_D3.0mm_L8.0mm_Horizontal_1EP_style1"
 			(at 92.71 101.6 0)
 			(effects

Commit message: pcb drawing continue..
Parts:
- removed Y2: 32.768Khz, Crystal:Crystal_C38-LF_D3.0mm_L8.0mm_Horizontal_1EP_style1, symbol Device:Crystal
- added Y3: 32.768Khz, Crystal:Crystal_C38-LF_D3.0mm_L8.0mm_Horizontal_1EP_style1, symbol Device:Crystal_GND3
Connections:
- net GND: now also Y3.3
- net at C54.2, U2.2 (OSCO): now also Y3.2
- net at C53.2, U2.1 (OSCI): now also Y3.1
Other:
- moved on the sheet: C54
Changed lines of the file:
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@@
 	(wire
 		(pts
-			(xy 76.2 110.49) (xy 77.47 110.49)
+			(xy 66.04 110.49) (xy 69.85 110.49)
 		)
 		(stroke
@@
 	(wire
 		(pts
+			(xy 86.36 101.6) (xy 87.63 101.6)
+		)
+		(stroke
+			(width 0)
+			(type default)
+		)
+	)
+	(wire
+		(pts
 			(xy 222.25 110.49) (xy 222.25 113.03)
 		)
@@
 	(wire
 		(pts
-			(xy 85.09 110.49) (xy 92.71 110.49)
+			(xy 77.47 110.49) (xy 92.71 110.49)
 		)
 		(stroke
@@
 	(symbol
 		(lib_id "Device:C")
-		(at 81.28 110.49 90)
+		(at 73.66 110.49 90)
 		(unit 1)
 		(exclude_from_sim no)
@@
 		(fields_autoplaced yes)
 		(property "Reference" "C54"
-			(at 81.28 100.33 90)
+			(at 73.66 100.33 90)
 			(effects
 				(font
@@
 		)
 		(property "Value" "15pF"
-			(at 81.28 102.87 90)
+			(at 73.66 102.87 90)
 			(effects
 				(font
@@
 		)
 		(property "Footprint" "Capacitor_SMD:C_0603_1608Metric"
-			(at 85.09 109.5248 0)
+			(at 77.47 109.5248 0)
 			(effects
 				(font
@@
 		)
 		(property "Datasheet" "~"
-			(at 81.28 110.49 0)
+			(at 73.66 110.49 0)
 			(effects
 				(font
@@
 		)
 		(property "Description" "Unpolarized capacitor"
-			(at 81.28 110.49 0)
+			(at 73.66 110.49 0)
 			(effects
 				(font
@@
 		)
 		(property "Package" "C0603"
-			(at 81.28 105.41 90)
+			(at 73.66 105.41 90)
 			(effects
 				(font
@@
 	)
 	(symbol
+		(lib_id "Device:Crystal_GND3")
+		(at 92.71 101.6 270)
+		(unit 1)
+		(exclude_from_sim no)
+		(in_bom yes)
+		(on_board yes)
+		(dnp no)
+		(fields_autoplaced yes)
+		(property "Reference" "Y3"
+			(at 96.52 100.3299 90)
+			(effects
+				(font
+					(size 1.27 1.27)
+				)
+				(justify left)
+			)
+		)
+		(property "Value" "32.768Khz"
+			(at 96.52 102.8699 90)
+			(effects
+				(font
+					(size 1.27 1.27)
+				)
+				(justify left)
+			)
+		)
+		(property "Footprint" "Crystal:Crystal_C38-LF_D3.0mm_L8.0mm_Horizontal_1EP_style1"
+			(at 92.71 101.6 0)
+			(effects
+				(font
+					(size 1.27 1.27)
+				)
+				(hide yes)
+			)
+		)
+		(property "Datasheet" "~"
+			(at 92.71 101.6 0)
+			(effects
+				(font
+					(size 1.27 1.27)
+				)
+				(hide yes)
+			)
+		)
+		(property "Description" "Three pin crystal, GND on pin 3"
+			(at 92.71 101.6 0)
+			(effects
+				(font
+					(size 1.27 1.27)
+				)
+				(hide yes)
+			)
+		)
+		(pin "3"
+		)
+		(pin "2"
+		)
+		(pin "1"
+		)
+		(instances
+			(project ""
+				(path "/1c1d47d5-f6ab-48f4-aef9-e333cdfe2713/c254b1ee-5d80-44f4-b3d6-0ba2c07a68ad"
+					(reference "Y3")
+					(unit 1)
+				)
+			)
+		)
+	)
+	(symbol
 		(lib_id "power:GND")
-		(at 76.2 110.49 270)
+		(at 66.04 110.49 270)
 		(unit 1)
 		(exclude_from_sim no)
@@
 		(fields_autoplaced yes)
 		(property "Reference" "#PWR0127"
-			(at 69.85 110.49 0)
+			(at 59.69 110.49 0)
 			(effects
 				(font
@@
 		)
 		(property "Value" "GND"
-			(at 72.39 110.4899 90)
+			(at 62.23 110.4899 90)
 			(effects
 				(font
@@
 		)
 		(property "Footprint" ""
-			(at 76.2 110.49 0)
+			(at 66.04 110.49 0)
 			(effects
 				(font
@@
 		)
 		(property "Datasheet" ""
-			(at 76.2 110.49 0)
+			(at 66.04 110.49 0)
 			(effects
 				(font
@@
 		)
 		(property "Description" "Power symbol creates a global label with name \"GND\" , ground"
-			(at 76.2 110.49 0)
+			(at 66.04 110.49 0)
 			(effects
 				(font
@@
 	)
 	(symbol
+		(lib_id "power:GND")
+		(at 86.36 101.6 270)
+		(unit 1)
+		(exclude_from_sim no)
+		(in_bom yes)
+		(on_board yes)
+		(dnp no)
+		(fields_autoplaced yes)
+		(property "Reference" "#PWR0175"
+			(at 80.01 101.6 0)
+			(effects
+				(font
+					(size 1.27 1.27)
+				)
+				(hide yes)
+			)
+		)
+		(property "Value" "GND"
+			(at 82.55 101.5999 90)
+			(effects
+				(font
+					(size 1.27 1.27)
+				)
+				(justify right)
+			)
+		)
+		(property "Footprint" ""
+			(at 86.36 101.6 0)
+			(effects
+				(font
+					(size 1.27 1.27)
+				)
+				(hide yes)
+			)
+		)
+		(property "Datasheet" ""
+			(at 86.36 101.6 0)
+			(effects
+				(font
+					(size 1.27 1.27)
+				)
+				(hide yes)
+			)
+		)
+		(property "Description" "Power symbol creates a global label with name \"GND\" , ground"
+			(at 86.36 101.6 0)
+			(effects
+				(font
+					(size 1.27 1.27)
+				)
+				(hide yes)
+			)
+		)
+		(pin "1"
+		)
+		(instances
+			(project "ea01"
+				(path "/1c1d47d5-f6ab-48f4-aef9-e333cdfe2713/c254b1ee-5d80-44f4-b3d6-0ba2c07a68ad"
+					(reference "#PWR0175")
+					(unit 1)
+				)
+			)
+		)
+	)
+	(symbol
 		(lib_id "Connector:TestPoint")
 		(at 153.67 99.06 180)
@@
 					(unit 1)
 				)
-			)
-		)
-	)
-	(symbol
-		(lib_id "Device:Crystal")
-		(at 92.71 101.6 90)
-		(unit 1)
-		(exclude_from_sim no)
-		(in_bom yes)
-		(on_board yes)
-		(dnp no)
-		(fields_autoplaced yes)
-		(property "Reference" "Y2"
-			(at 96.52 100.3299 90)
-			(effects
-				(font
-					(size 1.27 1.27)
-				)
-				(justify right)
-			)
-		)
-		(property "Value" "32.768Khz"
-			(at 96.52 102.8699 90)
-			(effects
-				(font
-					(size 1.27 1.27)
-				)
-				(justify right)
-			)
-		)
-		(property "Footprint" "Crystal:Crystal_C38-LF_D3.0mm_L8.0mm_Horizontal_1EP_style1"
-			(at 92.71 101.6 0)
-			(effects
-				(font
-					(size 1.27 1.27)
-				)
-				(hide yes)
-			)
-		)
-		(property "Datasheet" "~"
-			(at 92.71 101.6 0)
-			(effects
-				(font
-					(size 1.27 1.27)
-				)
-				(hide yes)
-			)
-		)
-		(property "Description" "Two pin crystal"
-			(at 92.71 101.6 0)
-			(effects
-				(font
-					(size 1.27 1.27)
-				)
-				(hide yes)
-			)
-		)
-		(pin "2"
-		)
-		(pin "1"
-		)
-		(instances
-			(project "ea01"
-				(path "/1c1d47d5-f6ab-48f4-aef9-e333cdfe2713/c254b1ee-5d80-44f4-b3d6-0ba2c07a68ad"
-					(reference "Y2")
-					(unit 1)
-				)

Commit message: component placement continue..
Parts:
- removed TP2, TP3, TP4, TP5: TestPoint, TestPoint:TestPoint_Pad_D1.5mm, symbol Connector:TestPoint

Commit message: placement continue...
Parts:
- removed C56: 22pF, Capacitor_SMD:C_0603_1608Metric, symbol Device:C
- removed TP1: TestPoint, TestPoint:TestPoint_Pad_D1.5mm, symbol Connector:TestPoint
- D16, D17: footprint Diode_SMD:D_SMA -> Diode_SMD:D_MiniMELF
Other:
- moved on the sheet: C55
