File: hw/ea01/power.kicad_sch (KiCad schematic)
At the start: 50 parts, among them J1 Screw_Terminal_01x02, U10 AMS1117-3.3, U4 MC34063AD, U5 AMS1117-5.0, U6 AMS1117-3.3, U7 MCP601-xOT

Commit message: errors fix for comp fp
Parts:
- J1: footprint TerminalBlock_RND:TerminalBlock_RND_205-00232_1x02_P5.08mm_Horizontal -> TerminalBlock:TerminalBlock_bornier-2_P5.08mm
Changed lines of the file:
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@@
 			)
 		)
-		(property "Footprint" "TerminalBlock_RND:TerminalBlock_RND_205-00232_1x02_P5.08mm_Horizontal"
+		(property "Footprint" "TerminalBlock:TerminalBlock_bornier-2_P5.08mm"
 			(at 22.86 35.56 0)
 			(effects

Commit message: component placement continue..
Parts:
- removed C17, C18, C21, C24, C35, C38: 10uF, Capacitor_THT:CP_Radial_D6.3mm_P2.50mm, symbol Device:C_Polarized
- removed C3: 100uF, Capacitor_THT:CP_Radial_D6.3mm_P2.50mm, symbol Device:C_Polarized
- removed D3: SMAJ24A, Diode_SMD:D_SMA, symbol Diode:SMAJ24A
- removed D4: RED_LED, Resistor_SMD:R_0805_2012Metric, symbol Device:LED
- removed FL1: Choke_CommonMode_FerriteCore_1234, Transformer_THT:Transformer_Toroid_Horizontal_D10.5mm_Amidon-T37, symbol Filter:Choke_CommonMode_FerriteCore_1234
- added C17, C18, C21, C24, C3, C35, C64: 10uF, Capacitor_SMD:C_0805_2012Metric, symbol Device:C
- added J19: Conn_01x02_Pin, Connector_PinHeader_2.54mm:PinHeader_1x02_P2.54mm_Vertical, symbol Connector:Conn_01x02_Pin
Connections:
- net +12V: now also C3.1
- net +3.3V: now also C18.1
- net +5V: now also C21.1
- net +6.8V: now also C17.1
- net 5V: now also C64.1
- net GND: now also D6.2 (A2), J1.1 (Pin_1), C17.2, C18.2, C21.2, C24.2, C3.2, C35.2, C64.2, J19.1 (Pin_1)
- net VBUS: now also C35.1
- net at C37.1, D1.2 (A), U10.2 (VO): now also C24.1
- net at D6.1 (A1), J1.2 (Pin_2): now also D5.2 (A)
- net at R11.2: now also J19.2 (Pin_2)

Commit message: placement continue...
Parts:
- removed C14, C15, C16, C37: 220nF, Capacitor_SMD:C_0603_1608Metric, symbol Device:C
- removed C24: 10uF, Capacitor_SMD:C_0805_2012Metric, symbol Device:C
- removed D1: SS26, Diode_SMD:D_SMA, symbol Diode:SS26
- removed R10, R7, R8: 10K, Resistor_SMD:R_0603_1608Metric, symbol Device:R
- removed R9: 100R, Resistor_SMD:R_0603_1608Metric, symbol Device:R
- removed U10: AMS1117-3.3, Package_TO_SOT_SMD:SOT-223-3_TabPin2, symbol Regulator_Linear:AMS1117-3.3
- removed U7: MCP601-xOT, Package_TO_SOT_SMD:SOT-23-5, symbol Amplifier_Operational:MCP601-xOT
- added J7: Conn_01x03_Pin, Connector_PinHeader_2.54mm:PinHeader_1x03_P2.54mm_Vertical, symbol Connector:Conn_01x03_Pin
Connections:
- net +5V: now also J7.2 (Pin_2)
- net VBUS: now also J7.3 (Pin_3)
- net 5V renamed +5V_REG
- net +5V_REG: now also J7.1 (Pin_1)
Other:
- moved on the sheet: C35, C36

Commit message: placement optimization and review continue
Parts:
- J19: footprint Connector_PinHeader_2.54mm:PinHeader_1x02_P2.54mm_Vertical -> Connector_PinHeader_1.27mm:PinHeader_1x02_P1.27mm_Vertical
Changed lines of the file:
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@@
 			)
 		)
-		(property "Footprint" "Connector_PinHeader_2.54mm:PinHeader_1x02_P2.54mm_Vertical"
+		(property "Footprint" "Connector_PinHeader_1.27mm:PinHeader_1x02_P1.27mm_Vertical"
 			(at 160.02 175.26 0)
 			(effects

Commit message: placement completed.
Parts:
- removed C17, C64: 10uF, Capacitor_SMD:C_0805_2012Metric, symbol Device:C
- removed C19, C20: 220nF, Capacitor_SMD:C_0603_1608Metric, symbol Device:C
- removed U5: AMS1117-5.0, Package_TO_SOT_SMD:SOT-223-3_TabPin2, symbol Regulator_Linear:AMS1117-5.0
Connections:
- net +6.8V is gone; now on net +5V_REG: C11.1, C12.1, C13.1, C9.1, L1.2, R6.1
- net GND: now also J1.2 (Pin_2); no longer J1.1 (Pin_1)
- net at D5.2 (A), D6.1 (A1): now also J1.1 (Pin_1); no longer J1.2 (Pin_2)
Other:
- moved on the sheet: C18, C21, C22, C23, C35, C36, D6, J1, J7, U6
