File: hw/ea01/ea01.kicad_pcb (KiCad board)
At the start: 2 copper layers, 100 x 45 mm, 194 parts, among them J1 Screw_Terminal_01x02, J10 Screw_Terminal_01x02, J11 Screw_Terminal_01x02, J12 Screw_Terminal_01x03, J13 Conn_01x02_Pin, J14 Conn_01x02_Pin, J15 Conn_01x02_Pin, J16 Conn_01x02_Pin, J17 Conn_01x02_Pin, J18 Conn_01x02_Pin, J19 Conn_01x02_Pin, J2 USB_B, J3 Conn_01x05_Pin, J4 Screw_Terminal_01x02, J5 Screw_Terminal_01x02, J6 Conn_01x02_Pin, J7 Conn_01x03_Pin, J8 Conn_01x03_Pin, J9 Conn_01x03_Pin, K1 G5NB, K2 G5NB, Q1 BC817, Q11 BC817, Q2 BC817, Q3 BC817, Q4 BC817, Q5 BC817, Q6 BC817, Q7 BC817, Q9 BC817, SW1 SW_Push, SW2 SW_Push, SW3 SW_Push, SW4 SW_Push, U1 RP2040, U11 W25Q32JVSS, U12 SN75176AP, U13 PC817, U14 PC817, U2 PCF8563T, U4 MC34063AD, U6 AMS1117-3.3, U8 CAT24C256, U9 74HC14, Y1 12Mhz, Y3 32.768Khz

Commit message: drawing continue...
Parts:
- removed C60: 100nF, Capacitor_SMD:C_0603_1608Metric
- removed C61: 22pF, Capacitor_SMD:C_0603_1608Metric
- removed J9: Conn_01x03_Pin, Connector_PinHeader_2.54mm:PinHeader_1x03_P2.54mm_Vertical
- removed R58: 1K, Resistor_SMD:R_0603_1608Metric
- C44, C52, C53, C54, R26, R29, R32, R35, R38, R39, R45, R55: moved to B.Cu
- moved R35 26.4 mm to (112.5, 54.6), turned to 180 degrees
- moved R32 24.6 mm to (112.5, 56.1), turned to 180 degrees
- moved R29 14.5 mm to (111.2, 60.6)
- moved R26 14.4 mm to (111.2, 59.1)
- moved C44 9.99 mm to (123.0, 58.0)
- moved R45 7.09 mm to (123.0, 59.5)
- moved C27 7.07 mm to (135.8, 57.7)
- moved J7 6.74 mm to (155.8, 76.8), turned to 180 degrees
- moved J8 5.11 mm to (147.7, 54.8), turned to -90 degrees
- moved C52 4.50 mm to (120.0, 58.0)
- moved R55 4.50 mm to (120.0, 59.5)
- moved C28 4.29 mm to (131.5, 62.7), turned to 0 degrees
- moved C30 3.26 mm to (125.8, 64.8), turned to 90 degrees
- moved R21 3.00 mm to (111.1, 60.6)
- moved U9 2.55 mm to (111.2, 66.9)
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Connections:
- U1 pad 13: unconnected-(U1-GPIO10-Pad13) -> OUT1_LED
- U1 pad 14: unconnected-(U1-GPIO11-Pad14) -> OUT0_LED
- U1 pad 36: OUT1_LED -> unconnected-(U1-GPIO24-Pad36)
- U1 pad 37: OUT0_LED -> unconnected-(U1-GPIO25-Pad37)
- U1 pad 38: VIN_MONITOR -> /mcu/HW_ADDRESS
- U1 pad 39: /mcu/ADC_TEST -> unconnected-(U1-GPIO27_ADC1-Pad39)
- U1 pad 41: /mcu/HW_ADDRESS -> unconnected-(U1-GPIO29_ADC3-Pad41)
Routing:
- net I2C0_SCL: track 0.00 -> 30.7 mm, vias 0 -> 3
- net /mcu/UART0_RX: track 0.00 -> 28.2 mm, vias 0 -> 1
- net I2C0_SDA: track 0.00 -> 28.0 mm, vias 0 -> 3
- net /mcu/UART0_TX: track 0.00 -> 25.9 mm, vias 0 -> 1
- net /mcu/HW_VER0: track 0.00 -> 21.4 mm, vias 0 -> 1
- net Net-(J3-Pin_1): track 0.00 -> 21.3 mm, vias 0 -> 1
- net /mcu/HW_VER1: track 1.50 -> 21.9 mm, vias 0 -> 1
- net IN1_LED: track 0.00 -> 20.1 mm, vias 0 -> 1
- net Net-(J3-Pin_2): track 0.00 -> 20.0 mm, vias 0 -> 1
- net OUT1_LED: track 0.00 -> 19.5 mm, vias 0 -> 1
- net OUT0_LED: track 0.00 -> 19.3 mm, vias 0 -> 1
- net /mcu/RUN: track 45.9 -> 64.4 mm, vias 0 -> 1
- net IN0_LED: track 0.00 -> 18.1 mm, vias 0 -> 1
- net RTC_INT: track 0.00 -> 16.5 mm
- net VBUS: track 5.81 -> 21.4 mm
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Other:
- board text added: "T R G"
- board text removed: "G R T"

Commit message: drawing continue..
Parts:
- removed D8: 1N4148W, Diode_SMD:D_SOD-123
- removed J6: Conn_01x02_Pin, Connector_PinHeader_1.27mm:PinHeader_1x02_P1.27mm_Vertical
- removed Q1: BC817, Package_TO_SOT_SMD:SOT-23
- removed R18, R19: 100R, Resistor_SMD:R_0603_1608Metric
- removed R20: 10K, Resistor_SMD:R_0603_1608Metric
- removed U9: 74HC14, Package_SO:SOIC-14_3.9x8.7mm_P1.27mm
- added U3: 74HC14, Package_SO:SOIC-14_3.9x8.7mm_P1.27mm, F.Cu at (111.3, 66.9)
- C45, FB5, FB6: moved to B.Cu
- moved R56 7.74 mm to (138.8, 71.1), turned to -90 degrees
- moved D6 7.60 mm to (133.0, 89.2), turned to 90 degrees
- moved C49 4.90 mm to (155.8, 80.1)
- moved R52 4.90 mm to (155.8, 81.6)
- moved C18 1.65 mm to (142.7, 76.8)
- moved C22 1.65 mm to (140.7, 80.5)
- moved C23 1.65 mm to (140.7, 76.8)
- moved C21 1.65 mm to (142.7, 80.5)
- moved Q4 0.64 mm to (103.1, 55.4)
- moved R22 0.64 mm to (102.9, 58.8)
- moved R27 0.64 mm to (105.8, 55.4)
- moved R33 0.64 mm to (105.8, 51.9)
- moved Q2 0.64 mm to (105.6, 58.8)
- moved Q3 0.61 mm to (105.6, 58.8)
- moved Q5 0.61 mm to (103.1, 55.4)
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Connections:
- U1 pad 18: BUZZER -> unconnected-(U1-GPIO15-Pad18)
Routing:
- net +3.3V: track 91.6 -> 305.3 mm, vias 13 -> 20
- net +12V: track 0.00 -> 76.9 mm, vias 0 -> 3
- net +5V_REG: track 0.00 -> 66.9 mm
- net Net-(C51-Pad1): track 0.00 -> 57.6 mm, vias 0 -> 1
- net Net-(C49-Pad1): track 0.00 -> 49.4 mm, vias 0 -> 1
- net +5V: track 0.00 -> 25.0 mm, vias 0 -> 4
- net Net-(D2-K): track 0.00 -> 14.1 mm
- net unconnected-(U1-GPIO15-Pad18): track 0.00 -> 11.9 mm
- net BUZZER: track 11.9 -> 0.00 mm
- net Net-(D5-A): track 0.00 -> 11.0 mm
- net +12V_RELAY: track 7.00 -> 17.6 mm
- net Net-(J3-Pin_1): track 21.3 -> 31.8 mm
- net Net-(Q2-B): track 1.84 -> 10.9 mm, vias 0 -> 2
- net /mcu/UDB_D+: track 22.4 -> 30.8 mm
- net /mcu/USB_D-: track 21.7 -> 30.1 mm
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- added copper zone on F.Cu, net +12V
- added copper zone on F.Cu, net Net-(U4-DC)

Commit message: drawing continue..
Parts:
- added C14: 220nF, Capacitor_SMD:C_0603_1608Metric, B.Cu at (141.7, 58.8)
- added C15: 220nF, Capacitor_SMD:C_0603_1608Metric, F.Cu at (136.8, 57.3)
- added R9: 100R, Resistor_SMD:R_0603_1608Metric, F.Cu at (136.0, 59.8)
- added U5: MCP9700Ax-ELT, Package_TO_SOT_SMD:SOT-353_SC-70-5, F.Cu at (138.2, 59.6)
- moved C43 1.72 mm to (105.7, 66.1)
- moved C47 1.72 mm to (105.7, 63.1)
- moved R44 1.72 mm to (104.2, 66.1)
- moved R50 1.72 mm to (104.2, 63.1)
- moved C25 1.36 mm to (127.8, 55.7), turned to 180 degrees
- moved R59 1.07 mm to (132.4, 56.0)
- moved C27 1.04 mm to (135.4, 56.7), turned to -90 degrees
- moved R21 0.95 mm to (111.1, 59.7)
- moved R23 0.95 mm to (111.1, 58.2)
- moved C10 0.85 mm to (130.6, 55.7)
- moved R82 0.40 mm to (136.2, 59.5)
- moved C32 0.15 mm to (128.0, 62.4)
- moved C34 0.15 mm to (128.0, 60.9)
- turned R67 to 90 degrees
- renumbered J12 to J6
Connections:
- FB4 pad 1: Net-(J12-Pin_3) -> unconnected-(FB4-Pad1)
- J6 pad 3: Net-(J12-Pin_3) -> unconnected-(FB4-Pad1)
- U1 pad 39: unconnected-(U1-GPIO27_ADC1-Pad39) -> BOARD_TEMP
- U3 pad 12: (no net) -> unconnected-(U3-Pad12)
- U3 pad 13: (no net) -> GND
- U3 pad 3: (no net) -> GND
- U3 pad 4: (no net) -> unconnected-(U3-Pad4)
Routing:
- net OUT1: track 2.00 -> 62.5 mm, vias 1 -> 2
- net OUT0: track 2.25 -> 55.6 mm, vias 1 -> 2
- net GND_RELAY: track 9.06 -> 52.7 mm, vias 0 -> 10
- net Net-(R49-Pad2): track 0.00 -> 38.2 mm, vias 0 -> 2
- net GND: track 0.04 -> 35.5 mm, vias 0 -> 39
- net Net-(R43-Pad2): track 0.00 -> 29.5 mm, vias 0 -> 2
- net RS485_TX: track 5.17 -> 33.3 mm, vias 0 -> 1
- net RS485_RW: track 6.26 -> 30.1 mm, vias 0 -> 1
- net RS485_RX: track 5.57 -> 27.5 mm, vias 0 -> 1
- net IN0_LED: track 18.1 -> 35.7 mm
- net IN1_LED: track 19.5 -> 35.2 mm
- net Net-(R55-Pad1): track 5.67 -> 17.9 mm, vias 0 -> 1
- net unconnected-(U1-GPIO15-Pad18): track 11.9 -> 0.00 mm
- net +3.3V: track 305.3 -> 315.1 mm, vias 20 -> 21
- net Net-(R45-Pad1): track 8.45 -> 17.9 mm, vias 0 -> 1
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
Commit message: draw contleted. Not checked yet.
Parts:
- added D1: NUP2105L, Package_TO_SOT_SMD:SOT-23, F.Cu at (150.8, 59.0)
- C45: moved to F.Cu
- moved C11 6.01 mm to (124.0, 91.6), turned to -90 degrees
- moved C45 4.18 mm to (106.6, 69.3), turned to 90 degrees
- moved R40 3.95 mm to (75.4, 78.2)
- moved R6 3.28 mm to (122.0, 91.6), turned to -90 degrees
- moved C42 2.05 mm to (75.4, 76.2)
- moved R42 2.05 mm to (75.4, 74.2)
- moved D14 0.98 mm to (75.0, 76.8)
- moved U6 0.55 mm to (141.7, 80.2)
- moved J19 0.35 mm to (128.4, 51.1)
- moved D15 0.25 mm to (75.0, 88.0)
- moved C15 0.15 mm to (136.7, 57.3)
- moved R41 0.15 mm to (75.4, 80.1)
Connections:
- net Net-(D18-A1) renamed /rs485/RS485_A
- net Net-(D19-A1) renamed /rs485/RS485_B
- FB4 pad 1: unconnected-(FB4-Pad1) -> /rs485/RS485_GND
- J6 pad 3: unconnected-(FB4-Pad1) -> /rs485/RS485_GND
Routing:
- net GND: track 35.5 -> 199.1 mm, vias 39 -> 109
- net Net-(D14-A2): track 0.00 -> 25.0 mm, vias 0 -> 1
- net Net-(D15-A2): track 0.00 -> 22.8 mm, vias 0 -> 1
- net /rs485/RS485_B: track 0.00 -> 18.3 mm
- net /rs485/RS485_A: track 0.00 -> 17.2 mm
- net +12V_RELAY: track 17.2 -> 28.8 mm
- net Net-(R42-Pad1): track 0.00 -> 8.33 mm, vias 0 -> 1
- net Net-(D15-A1): track 0.00 -> 7.58 mm, vias 0 -> 1
- net +3.3V: track 315.1 -> 321.5 mm, vias 21 -> 22
- net Net-(D14-A1): track 0.00 -> 6.29 mm, vias 0 -> 1
- net Net-(C42-Pad1): track 0.00 -> 6.04 mm
- net Net-(C46-Pad1): track 0.00 -> 6.03 mm
- net /rs485/RS485_GND: track 0.00 -> 6.00 mm
- net Net-(R48-Pad1): track 0.00 -> 4.54 mm
- net Net-(Q9-C): track 0.00 -> 3.71 mm
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- added copper zone on F.Cu, net +3.3V
- added copper zone on B.Cu, net /outputs/R0_A
- added copper zone on B.Cu, net /outputs/R0_B
- added copper zone on B.Cu, net /outputs/R1_A
- added copper zone on F.Cu, net /outputs/R1_A
- added copper zone on B.Cu, net /outputs/R1_B
- added copper zone on F.Cu, net /outputs/R1_B
- added copper zone on B.Cu, net GND
- added copper zone on F.Cu, net GND
Other:
- board text added: "+ -"
- board text added: "BOOT"
- board text added: "BT"
- board text added: "BT0"
- board text added: "BT1"
- board text added: "CDRVG"
- board text added: "ENIS ASLAN EA01-REV-A 2025"
- board text added: "EXT"
- board text added: "IN0"
- board text added: "IN0 -+"
- board text added: "IN1"
- board text added: "IN1 -+"
- board text added: "OUT0"
- board text added: "OUT1"
- board text added: "PLED"
- board text added: "R0"
- board text added: "R1"
- board text added: "RS485 A-B-G"
- board text added: "RUN"
- board text added: "U0"
- board text added: "U1"
- board text added: "USB"
