File: hw/ea01/outputs.kicad_sch (KiCad schematic)
At the start: 0 parts

Commit message: schmatic drawing continue...
Parts:
- added C62: 470uF, Capacitor_THT:CP_Radial_D8.0mm_P3.50mm, symbol Device:C_Polarized
- added D20, D21: SM4007, Diode_SMD:D_MELF, symbol Diode:SM4007
- added FB5, FB6: FerriteBead, symbol Device:FerriteBead
- added J10, J11: Screw_Terminal_01x02, TerminalBlock_RND:TerminalBlock_RND_205-00232_1x02_P5.08mm_Horizontal, symbol Connector:Screw_Terminal_01x02
- added K1, K2: SANYOU_SRD_Form_C, Relay_THT:Relay_SPDT_SANYOU_SRD_Series_Form_C, symbol Relay:SANYOU_SRD_Form_C
- added Q10, Q11, Q8, Q9: BC817, Package_TO_SOT_SMD:SOT-23, symbol Transistor_BJT:BC817
- added R69, R71, R74, R75, R78, R80: 100R, Resistor_SMD:R_0603_1608Metric, symbol Device:R
- added R70, R72, R73, R76, R77, R79: 10K, Resistor_SMD:R_0603_1608Metric, symbol Device:R
- added U15, U16: PC817, Package_DIP:DIP-4_W7.62mm, symbol Isolator:PC817
Connections:
- new net: J11.2 (Pin_2), K2.1
- new net: D21.2 (A), K2.2, R80.1
- new net: J11.1 (Pin_1), K2.3
- new net: Q11.3 (C), R80.2
- new net: Q10.1 (B), R75.2, R76.1
- new net: Q11.1 (B), R78.2, R79.1
- new net: Q9.1 (B), R69.2, R70.1
- new net: D20.2 (A), K1.2, R71.1
- new net: Q10.3 (C), U16.2
- new net: Q8.1 (B), R73.1, R74.2
- new net: Q8.3 (C), U15.2
- new net: R77.2, U16.1
- new net: J10.1 (Pin_1), K1.3
- new net: J10.2 (Pin_2), K1.1
- new net: R69.1, U15.3
- new net: R78.1, U16.3
- new net: Q9.3 (C), R71.2
- new net: R72.2, U15.1
- new net +12V: FB5.1
- new net +12V_RELAY: C62.1, D20.1 (K), D21.1 (K), FB5.2, K1.5, K2.5, U15.4, U16.4
- new net +5V: R72.1, R77.1
- new net GND: FB6.1, Q10.2 (E), Q8.2 (E), R73.2, R76.2
- new net GND_RELAY: C62.2, FB6.2, Q11.2 (E), Q9.2 (E), R70.2, R79.2
- new net OUT0: R74.1
- new net OUT1: R75.1

Commit message: errors fix for comp fp
Parts:
- FB5, FB6: footprint (none) -> Resistor_SMD:R_0805_2012Metric
- J10, J11: footprint TerminalBlock_RND:TerminalBlock_RND_205-00232_1x02_P5.08mm_Horizontal -> TerminalBlock:TerminalBlock_bornier-2_P5.08mm
Changed lines of the file:
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@@
 			)
 		)
-		(property "Footprint" "TerminalBlock_RND:TerminalBlock_RND_205-00232_1x02_P5.08mm_Horizontal"
+		(property "Footprint" "TerminalBlock:TerminalBlock_bornier-2_P5.08mm"
 			(at 200.66 113.03 0)
 			(effects
@@
 			)
 		)
-		(property "Footprint" ""
+		(property "Footprint" "Resistor_SMD:R_0805_2012Metric"
 			(at 36.83 123.698 90)
 			(effects
@@
 			)
 		)
-		(property "Footprint" "TerminalBlock_RND:TerminalBlock_RND_205-00232_1x02_P5.08mm_Horizontal"
+		(property "Footprint" "TerminalBlock:TerminalBlock_bornier-2_P5.08mm"
 			(at 200.66 33.02 0)
 			(effects
@@
 			)
 		)
-		(property "Footprint" ""
+		(property "Footprint" "Resistor_SMD:R_0805_2012Metric"
 			(at 38.1 100.838 90)
 			(effects

Commit message: pcb drawing continue..
Parts:
- removed K1, K2: SANYOU_SRD_Form_C, Relay_THT:Relay_SPDT_SANYOU_SRD_Series_Form_C, symbol Relay:SANYOU_SRD_Form_C
- added K1, K2: G5NB, Relay_THT:Relay_SPST_Omron_G5NB, symbol Relay:G5NB
Connections:
- net +12V_RELAY: now also K1.A1, K2.A1
- net at J11.2 (Pin_2): now also K2.13
- net at D21.2 (A), R80.1: now also K2.A2
- net at J11.1 (Pin_1): now also K2.14
- net at D20.2 (A), R71.1: now also K1.A2
- net at J10.1 (Pin_1): now also K1.14
- net at J10.2 (Pin_2): now also K1.13

Commit message: component placement continue..
Parts:
- removed Q10, Q8: BC817, Package_TO_SOT_SMD:SOT-23, symbol Transistor_BJT:BC817
- removed R72, R73, R76, R77: 10K, Resistor_SMD:R_0603_1608Metric, symbol Device:R
- removed R74, R75: 100R, Resistor_SMD:R_0603_1608Metric, symbol Device:R
- removed U15, U16: PC817, Package_DIP:DIP-4_W7.62mm, symbol Isolator:PC817
Connections:
- net OUT0: now also R69.1
- net OUT1: now also R78.1

Commit message: drawing continue...
Connections:
- net R1_A: now reaches J11.1 (Pin_1), K2.14
- net R1_B: now reaches J11.2 (Pin_2), K2.13
- net R0_A: now reaches J10.1 (Pin_1), K1.14
- net R0_B: now reaches J10.2 (Pin_2), K1.13
Changed lines of the file:
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@@
+		)
+	)
+	(label "R0_A"
+		(at 185.42 24.13 0)
+		(effects
+			(font
+				(size 1.27 1.27)
+			)
+			(justify left bottom)
+		)
+	)
+	(label "R1_B"
+		(at 185.42 124.46 0)
+		(effects
+			(font
+				(size 1.27 1.27)
+			)
+			(justify left bottom)
+		)
+	)
+	(label "R1_A"
+		(at 185.42 104.14 0)
+		(effects
+			(font
+				(size 1.27 1.27)
+			)
+			(justify left bottom)
+		)
+	)
+	(label "R0_B"
+		(at 185.42 44.45 0)
+		(effects
+			(font
+				(size 1.27 1.27)
+			)
+			(justify left bottom)
 		)
 	)
