File: hw/ea01/ea01.kicad_sch (KiCad schematic)
At the start: 0 parts

Commit message: schmatic drawing continue...
Other:
- added sheet buttons (buttons.kicad_sch)
Changed lines of the file:
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@@
+	)
+	(sheet
+		(at 95.25 60.96)
+		(size 27.94 12.7)
+		(exclude_from_sim no)
+		(in_bom yes)
+		(on_board yes)
+		(dnp no)
+		(fields_autoplaced yes)
+		(stroke
+			(width 0.1524)
+			(type solid)
+		)
+		(fill
+			(color 0 0 0 0.0000)
+		)
+		(property "Sheetname" "buttons"
+			(at 95.25 60.2484 0)
+			(effects
+				(font
+					(size 1.27 1.27)
+				)
+				(justify left bottom)
+			)
+		)
+		(property "Sheetfile" "buttons.kicad_sch"
+			(at 95.25 74.2446 0)
+			(effects
+				(font
+					(size 1.27 1.27)
+				)
+				(justify left top)
+			)
+		)
+		(instances
+			(project "ea01"
+				(path "/1c1d47d5-f6ab-48f4-aef9-e333cdfe2713"
+					(page "9")
+				)
+			)
+		)
 	)
 	(sheet

Commit message: drawing continue..
Other:
- added sheet temperature (temperature.kicad_sch)
Changed lines of the file:
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@@
+	)
+	(sheet
+		(at 95.25 81.28)
+		(size 26.67 11.43)
+		(exclude_from_sim no)
+		(in_bom yes)
+		(on_board yes)
+		(dnp no)
+		(fields_autoplaced yes)
+		(stroke
+			(width 0.1524)
+			(type solid)
+		)
+		(fill
+			(color 0 0 0 0.0000)
+		)
+		(property "Sheetname" "temperature"
+			(at 95.25 80.5684 0)
+			(effects
+				(font
+					(size 1.27 1.27)
+				)
+				(justify left bottom)
+			)
+		)
+		(property "Sheetfile" "temperature.kicad_sch"
+			(at 95.25 93.2946 0)
+			(effects
+				(font
+					(size 1.27 1.27)
+				)
+				(justify left top)
+			)
+		)
+		(instances
+			(project "ea01"
+				(path "/1c1d47d5-f6ab-48f4-aef9-e333cdfe2713"
+					(page "8")
+				)
+			)
+		)
 	)
 	(sheet
