File: hw/ea01/rs485.kicad_sch (KiCad schematic)
At the start: 1 part, among them U12 SN75176AP

Commit message: schmatic drawing continue...
Parts:
- added C58: 220nF, Capacitor_SMD:C_0603_1608Metric, symbol Device:C
- added C59: 1uF, Capacitor_SMD:C_0805_2012Metric, symbol Device:C
- added D18, D19: SMAJ12A, Diode_SMD:D_SMA, symbol Diode:SMAJ24A
- added FB4: FerriteBead, symbol Device:FerriteBead
- added J6: Screw_Terminal_01x03, symbol Connector:Screw_Terminal_01x03
- added J7: Conn_01x02_Pin, symbol Connector:Conn_01x02_Pin
- added R60: 120R, Resistor_SMD:R_1206_3216Metric, symbol Device:R
- added R61, R62: 47R, Resistor_SMD:R_0805_2012Metric, symbol Device:R
- added R63, R64: 4.7K, Resistor_SMD:R_0805_2012Metric, symbol Device:R
- added R65: 10K, Resistor_SMD:R_0603_1608Metric, symbol Device:R
- added R66, R67, R68: 100R, Resistor_SMD:R_0603_1608Metric, symbol Device:R
- added TP21, TP22: TestPoint, TestPoint:TestPoint_Pad_D1.5mm, symbol Connector:TestPoint
Connections:
- net at U12.1 (R): now also R68.1
- net at U12.2 (~{RE}): now also U12.3 (DE), R65.2, R66.1
- net at U12.4 (D): now also R67.1
- net GND: now reaches U12.5 (GND)
- net GND: now also C58.2, C59.2, D18.2 (A2), D19.2 (A2), FB4.2, R63.1, R65.1
- net at U12.6 (A): now also R62.2
- net at U12.7 (B): now also R61.1
- net +3.3V: now reaches U12.8 (VCC)
- net +3.3V: now also C58.1, C59.1, R64.1
- new net: D18.1 (A1), J6.1 (Pin_1), J7.1 (Pin_1), R62.1, R64.2, TP21.1
- new net: J7.2 (Pin_2), R60.2
- new net: D19.1 (A1), J6.2 (Pin_2), R60.1, R61.2, R63.2, TP22.1
- new net: FB4.1, J6.3 (Pin_3)
- new net RS485_RW: R66.2
- new net RS485_RX: R68.2
- new net RS485_TX: R67.2
Other:
- moved on the sheet: U12

Commit message: errors fix for comp fp
Parts:
- removed J6: Screw_Terminal_01x03, symbol Connector:Screw_Terminal_01x03
- added J12: Screw_Terminal_01x03, TerminalBlock:TerminalBlock_bornier-3_P5.08mm, symbol Connector:Screw_Terminal_01x03
- FB4: footprint (none) -> Resistor_SMD:R_0805_2012Metric
- J7: footprint (none) -> Connector_PinHeader_2.54mm:PinHeader_1x02_P2.54mm_Vertical
Connections:
- net at D18.1 (A1), J7.1 (Pin_1), R62.1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: now also J12.1 (Pin_1)
- net at D19.1 (A1), R60.1, R61.2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: now also J12.2 (Pin_2)
- net at FB4.1: now also J12.3 (Pin_3)
Other:
- moved on the sheet: C58, C59, D18, D19, FB4, J7, R60, R61, R62, R63, R64, R65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

Commit message: component placement continue..
Parts:
- removed J7: Conn_01x02_Pin, Connector_PinHeader_2.54mm:PinHeader_1x02_P2.54mm_Vertical, symbol Connector:Conn_01x02_Pin
- removed R60: 120R, Resistor_SMD:R_1206_3216Metric, symbol Device:R
- removed TP21, TP22: TestPoint, TestPoint:TestPoint_Pad_D1.5mm, symbol Connector:TestPoint

Commit message: drawing continue..
Parts:
- renumbered J12 to J6
Changed lines of the file:
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@@
 		(dnp no)
 		(fields_autoplaced yes)
-		(property "Reference" "J12"
+		(property "Reference" "J6"
 			(at 229.87 83.8199 0)
 			(effects
@@
 		(pin "3"
 		)
-		(instances
-			(project ""
-				(path "/1c1d47d5-f6ab-48f4-aef9-e333cdfe2713/6ca3256c-d43a-4bc8-af54-e996b7798b54"
-					(reference "J12")
-					(unit 1)
-				)
-			)
-		)
 	)

Commit message: draw contleted. Not checked yet.
Connections:
- net RS485_A: now reaches D18.1 (A1), J6.1 (Pin_1), R62.1, R64.2
- net RS485_B: now reaches D19.1 (A1), J6.2 (Pin_2), R61.2, R63.2
- net RS485_GND: now reaches FB4.1, J6.3 (Pin_3)
Other:
- moved on the sheet: FB4, J6
Changed lines of the file:
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@@
+	(wire
+		(pts
+			(xy 217.17 87.63) (xy 217.17 93.98)
+		)
+		(stroke
+			(width 0)
+			(type default)
+		)
+	)
 	(wire
 		(pts
@@
 	(wire
 		(pts
-			(xy 187.96 85.09) (xy 222.25 85.09)
+			(xy 187.96 85.09) (xy 229.87 85.09)
 		)
 		(stroke
@@
 	(wire
 		(pts
-			(xy 203.2 82.55) (xy 222.25 82.55)
+			(xy 203.2 82.55) (xy 229.87 82.55)
 		)
 		(stroke
@@
 	(wire
 		(pts
-			(xy 219.71 87.63) (xy 222.25 87.63)
-		)
-		(stroke
-			(width 0)
-			(type default)
-		)
-	)
-	(wire
-		(pts
 			(xy 83.82 86.36) (xy 86.36 86.36)
 		)
@@
 	(wire
 		(pts
+			(xy 229.87 87.63) (xy 217.17 87.63)
+		)
+		(stroke
+			(width 0)
+			(type default)
+		)
+	)
+	(wire
+		(pts
 			(xy 99.06 68.58) (xy 99.06 71.12)
 		)
@@
 	(wire
 		(pts
-			(xy 219.71 101.6) (xy 219.71 105.41)
-		)
-		(stroke
-			(width 0)
-			(type default)
-		)
-	)
-	(wire
-		(pts
-			(xy 219.71 93.98) (xy 219.71 87.63)
+			(xy 217.17 101.6) (xy 217.17 105.41)
 		)
 		(stroke
@@
 			(width 0)
 			(type default)
+		)
+	)
+	(label "RS485_GND"
+		(at 217.17 87.63 0)
+		(effects
+			(font
+				(size 1.27 1.27)
+			)
+			(justify left bottom)
+		)
+	)
+	(label "RS485_B"
+		(at 217.17 85.09 0)
+		(effects
+			(font
+				(size 1.27 1.27)
+			)
+			(justify left bottom)
+		)
+	)
+	(label "RS485_A"
+		(at 217.17 82.55 0)
+		(effects
+			(font
+				(size 1.27 1.27)
+			)
+			(justify left bottom)
 		)
 	)
@@
 	(symbol
 		(lib_id "Connector:Screw_Terminal_01x03")
-		(at 227.33 85.09 0)
+		(at 234.95 85.09 0)
 		(unit 1)
 		(exclude_from_sim no)
@@
 		(fields_autoplaced yes)
 		(property "Reference" "J6"
-			(at 229.87 83.8199 0)
+			(at 237.49 83.8199 0)
 			(effects
 				(font
@@
 		)
 		(property "Value" "Screw_Terminal_01x03"
-			(at 229.87 86.3599 0)
+			(at 237.49 86.3599 0)
 			(effects
 				(font
@@
 		)
 		(property "Footprint" "TerminalBlock:TerminalBlock_bornier-3_P5.08mm"
-			(at 227.33 85.09 0)
+			(at 234.95 85.09 0)
 			(effects
 				(font
@@
 		)
 		(property "Datasheet" "~"
-			(at 227.33 85.09 0)
+			(at 234.95 85.09 0)
 			(effects
 				(font
@@
 		)
 		(property "Description" "Generic screw terminal, single row, 01x03, script generated (kicad-library-utils/schlib/autogen/connector/)"
-			(at 227.33 85.09 0)
+			(at 234.95 85.09 0)
 			(effects
 				(font
@@
 	(symbol
 		(lib_id "power:GND")
-		(at 219.71 105.41 0)
+		(at 217.17 105.41 0)
 		(unit 1)
 		(exclude_from_sim no)
@@
 		(fields_autoplaced yes)
 		(property "Reference" "#PWR0147"
-			(at 219.71 111.76 0)
+			(at 217.17 111.76 0)
 			(effects
 				(font
@@
 		)
 		(property "Value" "GND"
-			(at 219.71 110.49 0)
+			(at 217.17 110.49 0)
 			(effects
 				(font
@@
 		)
 		(property "Footprint" ""
-			(at 219.71 105.41 0)
+			(at 217.17 105.41 0)
 			(effects
 				(font
@@
 		)
 		(property "Datasheet" ""
-			(at 219.71 105.41 0)
+			(at 217.17 105.41 0)
 			(effects
 				(font
@@
 		)
 		(property "Description" "Power symbol creates a global label with name \"GND\" , ground"
-			(at 219.71 105.41 0)
+			(at 217.17 105.41 0)
 			(effects
 				(font
@@
 	(symbol
 		(lib_id "Device:FerriteBead")
-		(at 219.71 97.79 0)
+		(at 217.17 97.79 0)
 		(unit 1)
 		(exclude_from_sim no)
@@
 		(fields_autoplaced yes)
 		(property "Reference" "FB4"
-			(at 223.52 96.4691 0)
+			(at 220.98 96.4691 0)
 			(effects
 				(font
@@
 		)
 		(property "Value" "FerriteBead"
-			(at 223.52 99.0091 0)
+			(at 220.98 99.0091 0)
 			(effects
 				(font
@@
 		)
 		(property "Footprint" "Resistor_SMD:R_0805_2012Metric"
-			(at 217.932 97.79 90)
+			(at 215.392 97.79 90)
 			(effects
 				(font
@@
 		)
 		(property "Datasheet" "~"
-			(at 219.71 97.79 0)
+			(at 217.17 97.79 0)
 			(effects
 				(font
@@
 		)
 		(property "Description" "Ferrite bead"
-			(at 219.71 97.79 0)
-			(effects
-				(font
+			(at 217.17 97.79 0)
+			(effects
+				(font
